File: VCM-addon-pcb.kicad_pcb (KiCad board)
At the start: 2 copper layers, 4 parts, among them U1 DRV8210DSGR

Commit message: add footprint lib
Parts:
- C2, C3, C4: footprint Capacitor_SMD:C_0603_1608Metric -> drv8210:C_0603_1608Metric
- U1: footprint footprints:DRV8210 -> drv8210:DRV8210
- moved C3 10.9 mm to (137.3, 104.5)
- moved C2 3.18 mm to (137.2, 107.0)
- moved C4 1.12 mm to (137.3, 111.5), turned to 180 degrees
Routing:
- net VCM +: track 0.00 -> 29.4 mm, vias 0 -> 2
- net SLEEP: track 0.00 -> 23.3 mm, vias 0 -> 1
- net VCM -: track 0.00 -> 17.5 mm, vias 0 -> 2
- net PWM_PH: track 0.00 -> 16.4 mm, vias 0 -> 1
- net PWM_EN: track 0.00 -> 14.1 mm, vias 0 -> 1
- net GNDREF: track 0.00 -> 13.0 mm, vias 0 -> 1
- net Net-(U1-VCC): track 0.00 -> 7.54 mm
- net unconnected-(C3-Pad1): track 0.00 -> 4.72 mm, vias 0 -> 1
- net Net-(U1-VM): track 0.00 -> 3.72 mm
- net Net-(U1-GND): track 0.00 -> 3.26 mm
- added copper zone on B.Cu, net GNDREF
- added copper zone on F.Cu, net GNDREF
Other:
- board outline added: 41 x 28 mm

Commit message: v0.1 schematic+pcb
Parts:
- added .54mm_Haaks: Header2.54mm_Haaks, Connector_PinHeader_2.54mm:PinHeader_1x06_P2.54mm_Horizontal, F.Cu at (136.6, 128.1)
- U1: value DRV8210DSGR -> DRV8210
Connections:
- C3 pad 1: unconnected-(C3-Pad1) -> Net-(U1-VCC)
Routing:
- net GNDREF: track 13.0 -> 58.6 mm
- net VCM -: track 17.5 -> 53.3 mm, vias 2 -> 3
- net VCM +: track 29.4 -> 50.9 mm, vias 2 -> 3
- net Net-(U1-VCC): track 7.54 -> 25.3 mm, vias 0 -> 1
- net PWM_PH: track 16.4 -> 33.6 mm
- net PWM_EN: track 14.1 -> 30.2 mm
- net SLEEP: track 23.3 -> 38.4 mm
- net unconnected-(C3-Pad1): track 4.72 -> 0.00 mm, vias 1 -> 0
Other:
- board size 41 x 28 mm -> 40.7 x 29.6 mm
- board text added: "VCM controller v0.1 (11-04-25)"
